File: pcb/fpga-gb-framebuffer.sch (KiCad schematic (older format))
At the start: 20 parts

Commit message: Updated PCB design
Connections:
- net IN_DATA_0: now also TinyFPGA_BX1.6 (Pin_6); no longer TinyFPGA_BX1.9 (Pin_9)
- net IN_DATA_1: now also TinyFPGA_BX1.8 (Pin_8); no longer TinyFPGA_BX1.10 (Pin_10)
- net IN_PIXEL_CLK: now also TinyFPGA_BX1.11 (Pin_11); no longer TinyFPGA_BX1.12 (Pin_12)
Changed lines of the file:
@@
 EESchema Schematic File Version 4
+LIBS:fpga-gb-framebuffer-cache
 EELAYER 26 0
 EELAYER END
@@
 Text GLabel 1600 5100 2    50   Output ~ 0
 IN_VSYNC
-Text GLabel 5150 1600 0    50   Input ~ 0
+Text GLabel 5150 1300 0    50   Input ~ 0
 IN_DATA_0
-Text GLabel 5150 1700 0    50   Input ~ 0
+Text GLabel 5150 1500 0    50   Input ~ 0
 IN_DATA_1
-Text GLabel 5150 1900 0    50   Input ~ 0
+Text GLabel 5150 1800 0    50   Input ~ 0
 IN_PIXEL_CLK
 Text GLabel 5150 2100 0    50   Input ~ 0

Commit message: Schematic update with tinyfpga symbol and pin assignment update for VGA
Parts:
- TinyFPGA_BX1: value Conn_02x14_Odd_Even -> FPGA; symbol Connector_Generic:Conn_02x14_Counter_Clockwise -> TinyFPGA_BX:TinyFPGA_BX
Connections:
- net OUT_B_0: now also TinyFPGA_BX1.19 (18); no longer TinyFPGA_BX1.20 (Pin_20)
- net OUT_B_1: now also TinyFPGA_BX1.18 (17); no longer TinyFPGA_BX1.19 (Pin_19)
- net OUT_G_0: now also TinyFPGA_BX1.22 (21); no longer TinyFPGA_BX1.23 (Pin_23)
- net OUT_G_1: now also TinyFPGA_BX1.21 (20); no longer TinyFPGA_BX1.22 (Pin_22)
- net OUT_R_0: now also TinyFPGA_BX1.25 (24); no longer TinyFPGA_BX1.26 (Pin_26)
- net OUT_R_1: now also TinyFPGA_BX1.24 (23); no longer TinyFPGA_BX1.25 (Pin_25)
- net VGA_HSYNC: now also TinyFPGA_BX1.16 (15); no longer TinyFPGA_BX1.17 (Pin_17)
Other:
- moved on the sheet: TinyFPGA_BX1
Changed lines of the file:
@@
 GB_DATA_1
 $Comp
-L Connector_Generic:Conn_02x14_Counter_Clockwise TinyFPGA_BX1
+L TinyFPGA_BX:TinyFPGA_BX TinyFPGA_BX1
 U 1 1 5C3BA172
 P 5350 1400
 F 0 "TinyFPGA_BX1" H 5400 2217 50  0000 C CNN
-F 1 "Conn_02x14_Odd_Even" H 5400 2126 50  0000 C CNN
+F 1 "FPGA" H 5400 2126 50  0000 C CNN
 F 2 "pcb:TinyFPGA_BX" H 5350 1400 50  0001 C CNN
 F 3 "~" H 5350 1400 50  0001 C CNN
@@
 	1    0    0    -1
 $EndComp
-Wire Wire Line
-	4650 600  4950 600
-Wire Wire Line
-	4950 600  4950 800
-Wire Wire Line
-	4950 800  5150 800
 $Comp
 L Connector:DB15_Female_HighDensity VGA1
@@
 Text GLabel 1600 5100 2    50   Output ~ 0
 IN_VSYNC
-Text GLabel 5150 1300 0    50   Input ~ 0
+Text GLabel 5000 1300 0    50   Input ~ 0
 IN_DATA_0
-Text GLabel 5150 1500 0    50   Input ~ 0
+Text GLabel 5000 1500 0    50   Input ~ 0
 IN_DATA_1
-Text GLabel 5150 1800 0    50   Input ~ 0
+Text GLabel 5000 1800 0    50   Input ~ 0
 IN_PIXEL_CLK
-Text GLabel 5150 2100 0    50   Input ~ 0
+Text GLabel 5000 2100 0    50   Input ~ 0
 IN_VSYNC
-Text GLabel 5650 1100 2    50   Output ~ 0
+Text GLabel 5700 1200 2    50   Output ~ 0
 OUT_R_1
-Text GLabel 5650 1300 2    50   Output ~ 0
+Text GLabel 5700 1400 2    50   Output ~ 0
 OUT_G_0
-Text GLabel 5650 1600 2    50   Output ~ 0
+Text GLabel 5700 1700 2    50   Output ~ 0
 OUT_B_0
-Text GLabel 5650 2100 2    50   Output ~ 0
+Text GLabel 5700 2100 2    50   Output ~ 0
 VGA_VSYNC
-Text GLabel 5650 1900 2    50   Output ~ 0
+Text GLabel 5700 2000 2    50   Output ~ 0
 VGA_HSYNC
 Text Notes 2900 1900 2    50   ~ 0
@@
 Text Notes 9500 2550 2    50   ~ 0
 FPGA 3.3v signal needs dividing and laddering for VGA RGB 0 - 0.7V signal
-Text GLabel 5650 1000 2    50   Output ~ 0
+Text GLabel 5700 1100 2    50   Output ~ 0
 OUT_R_0
-Text GLabel 5650 1400 2    50   Output ~ 0
+Text GLabel 5700 1500 2    50   Output ~ 0
 OUT_G_1
-Text GLabel 5650 1700 2    50   Output ~ 0
+Text GLabel 5700 1800 2    50   Output ~ 0
 OUT_B_1
 $Comp
@@
 Wire Wire Line
 	8950 3300 8750 3300
+Wire Wire Line
+	4650 600  5000 600
+Wire Wire Line
+	5000 600  5000 800
 $EndSCHEMATC
